File: Fiesta_pcbs/ecu/ECU/ECU.kicad_sch (KiCad schematic)
At the start: 76 parts, among them J1 VP37 connector, J2 Conn_01x01_Socket, J3 Conn_01x01_Socket, J4 Conn_01x01_Socket, J5 Conn_01x01_Socket, J6 Conn_01x01_Socket, J7 Conn_01x01_Socket, J8 Conn_01x01_Socket, J9 Conn_01x01_Socket, K1 G5V-2, Q1 BC547, Q10 BDW93, Q2 2SK107, Q3 BDW93, Q4 IRF540N, Q5 BDW93, Q6 BDW93, Q7 BDW93, Q8 BDW93, Q9 BDW93, U1 UA78M08, U2 RP2040-Zero, U3 L7805, U4 LM2931-3.3_TO220, U5 PCF8574AP

Commit message: feat(schems, legacy): refresh ECU KiCad project, add custom module libraries, and archive old legacy sketches
- update ECU schematic/project files and regenerate project PDF
- add custom KiCad footprint library (MCP2515, GY-NEO6MV2, OBD2 J1962)
- add matching KiCad symbol library entries
- remove obsolete legacy sources and replace them with archived zip bundles
- README update
- next release (1.1.0)
Parts:
- removed 100nF2: C_Small, symbol Device:C_Small
- removed 10K (x2), 10K1, 10K10, 10K11, 10K2, 10K3, 10K4, 10K5, 10K6, 10K7, 10K8: R_Small, symbol Device:R_Small
- removed 10uF1, 10uF2, 10uF3: C_Polarized, symbol Device:C_Polarized
- removed D3: D_Schottky_Dual_CommonCathode_AKA, symbol Device:D_Schottky_Dual_CommonCathode_AKA
- added 100R, 10K, 10k (x6), 1K (x9), 1k5 (x2), 1k7, 220R (x3), 2K2 (x2), 2k2 (x3), 3.3K, 47K (x3), 4k7 (x2), 51K, 51K1: R_Small, symbol Device:R_Small
- added 100nF (x8), 100nF1: C_Small, symbol Device:C_Small
- added 100uF (x4), 10uF, 1uF (x8), 2200uF (x2): C_Polarized, symbol Device:C_Polarized
- added 10A: Fuse, symbol Device:Fuse
- added D12, D13, D14, D26: 1N4003, Diode_THT:D_DO-41_SOD81_P10.16mm_Horizontal, symbol Diode:1N4003
- added D15, D16, D17, D18, D19, D20, D31: BAT48RL, Diode_THT:D_DO-35_SOD27_P7.62mm_Horizontal, symbol Diode:BAT48RL
- added D21, D23, D25: C3D16065A, Package_TO_SOT_THT:TO-220-2_Vertical, symbol Diode:C3D16065A
- added D22, D24, D3: 1N5818, Diode_THT:D_DO-41_SOD81_P10.16mm_Horizontal, symbol Diode:1N5818
- added D27, D28, D29, D30: SD05C-01F, Diode_SMD:D_SOD-323, symbol Diode:SD05C-01F
- added D33: ZY3.3V, Diode_THT:D_DO-41_SOD81_P10.16mm_Horizontal, symbol Diode:ZYxxx
- added J10, J11, J12, J13, J14, J15, J16, J17, J18, J19, J20, J21, J22, J23, J24, J25, J26, J27, J28, J29, J30, J31, J33, J34, J35, J36, J37, J38, J39, J40, J41, J42, J43, J44, J45, J46, J47, J48, J49: Conn_01x01_Socket, symbol Connector:Conn_01x01_Socket
- added J32: OBD2_J1962_Female_16P, FiestaFootprints:OBD2_J1962_Female_16P_Generic, symbol Fiesta_Modules:OBD2_J1962_Female_16P_Generic
- added Q11, Q12: 2N6037, Package_TO_SOT_THT:TO-220-3_Vertical, symbol Transistor_BJT:BDW93
- added Q13, Q14, Q17, Q19, Q21, Q23: BC547, Package_TO_SOT_THT:TO-92_Inline, symbol Transistor_BJT:BC547
- added Q15, Q18, Q22: BC557, Package_TO_SOT_THT:TO-92_Inline, symbol Transistor_BJT:BC557
- added Q16, Q20: IRF540N, Package_TO_SOT_THT:TO-220-3_Vertical, symbol Transistor_FET:IRF540N
- added U11: AMS1117-3.3, Package_TO_SOT_SMD:SOT-223-3_TabPin2, symbol Regulator_Linear:AMS1117-3.3
- added U6: 4051, symbol 4xxx:4051
- added U7, U8: MCP2515_CAN, FiestaFootprints:MCP2515_CAN_Module_7P54, symbol Fiesta_Modules:MCP2515_CAN_Module_7P54
- added U9: GY_NEO6MV2, FiestaFootprints:GY_NEO6MV2_Module_4P254, symbol Fiesta_Modules:GY_NEO6MV2_Module_4P254
- A1: value RaspberryPi_Pico -> RaspberryPi_Pico (RP2040)
- Q10, Q3, Q5, Q6, Q7, Q8, Q9: value BDW93 -> 2N6037
- U4: value LM2931-3.3_TO220 -> LM2931-3.3
Connections:
- net GND: now also Q4.3 (S), U5.8 (GND), 100nF.1, 100nF.1, 100nF.2, 100nF.2, 100nF.2, 100nF1.2, 100uF.2, 100uF.2, 100uF.2, 100uF.2, 10K.1, 10uF.2, 1uF.2, 1uF.2, 1uF.2, 1uF.2, 1uF.2, 1uF.2, 1uF.2, 1uF.2, 2200uF.2, 2200uF.2, 3.3K.2, D17.2 (A), D18.2 (A), D22.2 (A), D24.2 (A), D26.2 (A), D27.1 (A1), D28.1 (A1), D29.1 (A1), D3.2 (A), D30.1 (A1), J28.1 (Pin_1), J32.5 (SIGNAL_GND), J36.1 (Pin_1), J45.1 (Pin_1), J46.1 (Pin_1), J48.1 (Pin_1), J49.1 (Pin_1), Q11.3 (E), Q12.3 (E), Q13.3 (E), Q15.1 (C), Q16.3 (S), Q18.1 (C), Q19.3 (E), Q20.3 (S), Q22.1 (C), Q23.3 (E), U11.1 (GND), U6.6 (Inh), U6.7 (VEE), U6.8 (VSS), U7.2 (GND), U8.2 (GND), U9.4 (GND); no longer U5.16 (VDD)
- net at RN1.2 (R1), U5.4 (P0): now also 1K.2
- net at Q5.1 (B): now also 1K.1
- net at 10K.1, 10K.1, J1.2 (Pin_2)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: now also J15.1 (Pin_1)
- net at D10.1 (K), D2.2 (A), D4.1 (K)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: now also 100nF.1, 2200uF.1, 47K.2, D12.1 (K), D13.1 (K), D14.1 (K), D21.1 (K), D23.1 (K), D25.1 (K), D26.1 (K), J18.1 (Pin_1), J19.1 (Pin_1)
- net at 100nF.1, 10uF.1, A1.39 (VSYS)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: now also 100uF.1, J39.1 (Pin_1)
- net at 100nF.1, RN1.1 (common), U4.3 (VO): now also D1.2 (A), U5.16 (VDD), 100nF.1, 100nF.1, 100nF1.1, 100uF.1, 100uF.1, 10k.2, 10k.2, 10k.2, 1K.1, 1k5.1, 1k5.1, 2K2.1, 2K2.1, 2k2.2, 2k2.2, 2k2.2, 4k7.1, 4k7.1, 51K.1, 51K1.1, D15.1 (K), D16.1 (K), D31.2 (A), J40.1 (Pin_1), J44.1 (Pin_1), Q14.1 (C), Q17.1 (C), Q21.1 (C), U6.16 (VDD), U7.1 (VCC), U8.1 (VCC); no longer D1.1 (K), U5.8 (GND)
- net at Q4.1 (G): now also 220R.1
- net at Q4.2 (D): now also D21.2 (A), D22.1 (K), J17.1 (Pin_1)
- net at Q9.1 (B): now also 1K.1
- net at 100nF.1, 100nF.1, 47K.1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: now also 2200uF.1
- net at A1.34 (GPIO28_ADC2): now also 100nF.2, 10K.2, 47K.1
- net at 10nF.1, 10nF.2, J1.1 (Pin_1): now also J16.1 (Pin_1)
- net at A1.2 (GPIO1), U2.11 (GP1), U5.14 (SCL): now also 2K2.2, D29.2 (A2), J42.1 (Pin_1)
- net at RN1.3 (R2), U5.5 (P1): now also 1K.2
- net at Q6.1 (B): now also 1K.1
- net at D11.1 (K), J8.1 (Pin_1), K1.8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: now also J1.8 (Pin_8), D14.2 (A)
- net at 1uF.1, 3.3K.2, J1.7 (Pin_7)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: now also J14.1 (Pin_1)
- net at A1.1 (GPIO0), U2.10 (GP0), U5.15 (SDA): now also 2K2.2, D30.2 (A2), J43.1 (Pin_1)
- net at J1.10 (Pin_10): now also J1.5 (Pin_5), 10A.1
- net at J1.6 (Pin_6): now also D24.1 (K), D25.2 (A), J30.1 (Pin_1), Q20.2 (D)
- net at J1.9 (Pin_9): now also D23.2 (A), D3.1 (K), J31.1 (Pin_1), Q16.2 (D)
- net at A1.10 (GPIO7): now also D16.2 (A), D17.1 (K), D19.2 (A)
- net at A1.11 (GPIO8): now also 1K.2
- net at A1.12 (GPIO9): now also 100nF.1, 10k.1, 10k.2
- net at A1.14 (GPIO10): now also 100nF.1, 10k.1, 10k.2
- net at A1.15 (GPIO11): now also U6.11 (A)
- net at A1.16 (GPIO12): now also U6.10 (B)
- net at A1.17 (GPIO13): now also U6.9 (C)
- net at A1.19 (GPIO14): now also 4k7.2, U8.7 (INT)
- net at A1.20 (GPIO15): now also 4k7.2, U7.7 (INT)
- net at A1.21 (GPIO16): now also U7.4 (SO), U8.4 (SO)
- net at A1.22 (GPIO17): now also U7.3 (CS)
- net at A1.24 (GPIO18): now also U7.6 (SCK), U8.6 (SCK)
- net at A1.25 (GPIO19): now also U7.5 (SI), U8.5 (SI)
- net at A1.26 (GPIO20): now also 1K.2, 1uF.1, J41.1 (Pin_1)
- net at A1.27 (GPIO21): now also 47K.2, U9.3 (TX)
- net at A1.29 (GPIO22): now also 47K.2, U9.2 (RX)
- net at A1.32 (GPIO27_ADC1): now also U6.3 (X)
- net at A1.36 (3V3): now also D1.1 (K); no longer D1.2 (A)
- net at A1.4 (GPIO2): now also D15.2 (A), D18.1 (K), D20.2 (A)
- net at A1.7 (GPIO5): now also 100nF.1, 10k.1, 10k.2
- net at A1.9 (GPIO6): now also U8.3 (CS)
- net at Q3.1 (B): now also 1K.1
- net at Q7.1 (B): now also 1K.1
- net at RN1.7 (R6), U5.10 (P5): now also 1K.2
- net at RN1.8 (R7), U5.11 (P6): now also 1K.2
- net at RN1.4 (R3), U5.6 (P2): now also 1K.2
- net at RN1.5 (R4), U5.7 (P3): now also 1K.2
- net at RN1.6 (R5), U5.9 (P4): now also 1K.2
- net at Q8.1 (B): now also 1K.1
- new net: 1K.1, Q12.1 (B)
- new net: D13.2 (A), J11.1 (Pin_1), Q12.2 (C)
- new net: 2k2.1, Q17.2 (B), Q18.2 (B), Q19.1 (C)
- new net: 220R.2, Q17.3 (E), Q18.3 (E)
- new net: 1k5.2, 1uF.1, J21.1 (Pin_1), U6.14 (X1)
- new net: D20.1 (K), D27.2 (A2), J13.1 (Pin_1)
- new net: 2k2.1, Q13.1 (C), Q14.2 (B), Q15.2 (B)
- new net: 220R.2, Q14.3 (E), Q15.3 (E)
- new net: 1k7.1, J25.1 (Pin_1)
- new net: J32.14 (CAN_L), J34.1 (Pin_1), U8.8 (CANL)
- new net: J32.6 (CAN_H), J35.1 (Pin_1), U8.9 (CANH)
- new net: J38.1 (Pin_1), U7.8 (CANL)
- new net: J37.1 (Pin_1), U7.9 (CANH)
- new net: 2k2.1, Q21.2 (B), Q22.2 (B), Q23.1 (C)
- new net: 220R.2, Q21.3 (E), Q22.3 (E)
- new net: 100nF.2, 10k.1, Q23.2 (B)
- new net: 1uF.1, 47K.1, 47K.1, D31.1 (K), U11.2 (VO), U9.1 (VCC)
- new net: 10uF.1, D33.2 (A), U11.3 (VI)
- new net: 10A.2, J29.1 (Pin_1)
- new net: 220R.1, Q16.1 (G)
- new net: 1K.1, Q11.1 (B)
- new net: 1k5.2, 1uF.1, J20.1 (Pin_1), U6.13 (X0)
- new net: 100nF.2, 10k.1, Q13.2 (B)
- new net: D19.1 (K), D28.2 (A2), J12.1 (Pin_1)
- new net: 100nF.2, 1k7.2, 3.3K.1, U6.5 (X5)
- new net: 1uF.1, J26.1 (Pin_1), U6.2 (X6)
- new net: 1uF.1, J22.1 (Pin_1), U6.15 (X2)
- new net: 100nF.2, 10k.1, Q19.2 (B)
- new net: 1uF.1, J27.1 (Pin_1), U6.4 (X7)
- new net: 100R.1, 100uF.1, 51K1.2, J24.1 (Pin_1)
- new net: 100R.2, U6.1 (X4)
- new net: D12.2 (A), J10.1 (Pin_1), Q11.2 (C)
- new net: 1uF.1, 51K.2, J23.1 (Pin_1), U6.12 (X3)
- new net: 220R.1, Q20.1 (G)
- new net: D33.1 (K), J32.16 (VBAT_12V), J33.1 (Pin_1), J47.1 (Pin_1)
Other:
- note added: "+12V"
- note added: "+12V/BATT"
- note added: "+3.3V"
- note added: "1"
- note added: "100"
- note added: "12"
- note added: "12V"
- note added: "12V / IGN"
- note added: "13"
- note added: "14"
- note added: "15"
- note added: "16"
- note added: "17"
- note added: "19"
- note added: "21"
- note added: "22"
- note added: "24"
- note added: "25"
- note added: "27"
- note added: "3.3V"
- note added: "31"
- note added: "32"
- note added: "34"
- note added: "35"
- note added: "39"
- note added: "41"
- note added: "42"
- note added: "49"
- note added: "50"
- note added: "51"
- note added: "53"
- note added: "55"
- note added: "57"
- note added: "58"
- note added: "5V"
- note added: "63"
- note added: "66"
- note added: "68"
- note added: "69"
- note added: "70"
- note added: "71"
- note added: "76"
- note added: "77"
- note added: "8"
- note added: "80"
- note added: "83"
- note added: "92"
- note added: "96"
- note added: "97"
- note added: "A1"
- note added: "AIR TEMP"
- note added: "ANGLE"
- note added: "CAN"
- note added: "CAN-H"
- note added: "CAN-L"
- note added: "COOLANT TEMP"
- note added: "CS/CAN"
- note added: "CS/OBD-2"
- note added: "DPF LAMP"
- note added: "ENGINE HEAT HI"
- note added: "ENGINE HEAT LO"
- note added: "FAN"
- note added: "FUEL ON/OFF"
- note added: "FUEL TANK AMOUNT"
- note added: "FUEL TEMP"
- note added: "GLOW PLUGS"
- note added: "GLOW PLUGS LAMP"
- note added: "GND"
- note added: "GP10"
- note added: "GP2"
- note added: "GP5"
- note added: "GP7"
- note added: "GP8"
- note added: "GP9"
- note added: "H/WIND"
- note added: "H/WIND BUTTON"
- note added: "HALL"
- note added: "INJECTOR"
- note added: "INT/CAN"
- note added: "INT/OBD-2"
- note added: "MISO"
- note added: "MOSI"
- note added: "N/A"
- note added: "OBD-2"
- note added: "OBD-2 CAN-H"
- note added: "OBD-2 CAN-L"
- note added: "OIL TEMP"
- note added: "RX"
- note added: "SCK"
- note added: "THROTTLE"
- note added: "TURBO"
- note added: "TURBO PRESSURE"
- note added: "TX"
- note added: "VP37 ADJ"
- company: (none) -> Marcin Kielesiński PROFI-SOFT
- title: (none) -> Fiesta VP37 ECU
- moved on the sheet: 100K, 100nF, 10K, 10nF, 10uF, 1K, 1uF, 3.3K, 47K, 51K, A1, D1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

Commit message: feat(schem): circuit update (kicad / pdf)
Parts:
- added D32, D34, D35, D36: SD05C-01F, Diode_SMD:D_SOD-323, symbol Diode:SD05C-01F
Connections:
- net GND: now also D32.1 (A1), D34.1 (A1), D35.1 (A1), D36.1 (A1)
- net at J32.14 (CAN_L), J34.1 (Pin_1), U8.8 (CANL): now also D35.2 (A2)
- net at J32.6 (CAN_H), J35.1 (Pin_1), U8.9 (CANH): now also D36.2 (A2)
- net at J38.1 (Pin_1), U7.8 (CANL): now also D34.2 (A2)
- net at J37.1 (Pin_1), U7.9 (CANH): now also D32.2 (A2)
Other:
- moved on the sheet: J32
