File: Fiesta_pcbs/ecu/ECU/ECU.kicad_sch (KiCad schematic)
At the start: 204 parts, among them J1 VP37 connector, J10 Conn_01x01_Socket, J11 Conn_01x01_Socket, J12 Conn_01x01_Socket, J13 Conn_01x01_Socket, J14 Conn_01x01_Socket, J15 Conn_01x01_Socket, J16 Conn_01x01_Socket, J17 Conn_01x01_Socket, J18 Conn_01x01_Socket, J19 Conn_01x01_Socket, J2 Conn_01x01_Socket, J20 Conn_01x01_Socket, J21 Conn_01x01_Socket, J22 Conn_01x01_Socket, J23 Conn_01x01_Socket, J24 Conn_01x01_Socket, J25 Conn_01x01_Socket, J26 Conn_01x01_Socket, J27 Conn_01x01_Socket, J28 Conn_01x01_Socket, J29 Conn_01x01_Socket, J3 Conn_01x01_Socket, J30 Conn_01x01_Socket, J31 Conn_01x01_Socket, J32 OBD2_J1962_Female_16P, J33 Conn_01x01_Socket, J34 Conn_01x01_Socket, J35 Conn_01x01_Socket, J36 Conn_01x01_Socket, J37 Conn_01x01_Socket, J38 Conn_01x01_Socket, J39 Conn_01x01_Socket, J4 Conn_01x01_Socket, J40 Conn_01x01_Socket, J41 Conn_01x01_Socket, J42 Conn_01x01_Socket, J43 Conn_01x01_Socket, J44 Conn_01x01_Socket, J45 Conn_01x01_Socket, J46 Conn_01x01_Socket, J47 Conn_01x01_Socket, J48 Conn_01x01_Socket, J49 Conn_01x01_Socket, J5 Conn_01x01_Socket, J6 Conn_01x01_Socket, J7 Conn_01x01_Socket, J8 Conn_01x01_Socket, J9 Conn_01x01_Socket, K1 G5V-2, Q1 BC547, Q10 2N6037, Q11 2N6037, Q12 2N6037, Q13 BC547, Q14 BC547, Q15 BC557, Q16 IRF540N, Q17 BC547, Q18 BC557, Q19 BC547, Q2 2SK107, Q20 IRF540N, Q21 BC547, Q22 BC557, Q23 BC547, Q3 2N6037, Q4 IRF540N, Q5 2N6037, Q6 2N6037, Q7 2N6037, Q8 2N6037, Q9 2N6037, U1 UA78M08, U11 AMS1117-3.3, U2 RP2040-Zero, U3 L7805, U4 LM2931-3.3, U5 PCF8574AP, U6 4051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

Commit message: feat(ecu): refine VP37 control and feedback -Tune actuator response and prevent delayed rebound damping -Harden persistence and isolate host device tests -Update ECU hardware assets, tooling and docs
Connections:
- net at 100nF.1, 2200uF.1, 47K.2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: now also 2k2.2, 2k2.2, 2k2.2, Q14.1 (C), Q17.1 (C), Q21.1 (C)
- net at 100nF.1, 100nF.1, 100nF.1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: no longer 2k2.2, 2k2.2, 2k2.2, Q14.1 (C), Q17.1 (C), Q21.1 (C)
Other:
- moved on the sheet: 220R, D21, D27, D28

Commit message: fix(vp37): restore shunt travel and add passive sensing -Add current and full-period supply measurements. -Confirm settled position before holding the integral.
Parts:
- added 0.22R: R_Small, symbol Device:R_Small
- added D37: BZV55C3V3, Diode_SMD:D_MiniMELF, symbol Diode:BZV55C3V3
Connections:
- net GND: now also 0.22R.1, D37.2 (A); no longer Q20.3 (S)
- net at A1.31 (GPIO26_ADC0): now also Q20.3 (S), 0.22R.2, D37.1 (K)
Other:
- note added: "ADC0"
- note added: "CURRENT"
