File: Fiesta_pcbs/dashboard/Clocks/Clocks.kicad_sch (KiCad schematic)
At the start: 53 parts, among them J1 Conn_01x01_Pin, J2 Conn_01x05_Pin, J3 Conn_02x06_Odd_Even, J4 Conn_01x02_Pin, Q1 2N7000, Q2 BC307, Q3 ZTX601, Q4 ZTX601, Q5 ZTX601, Q6 ZTX601, Q7 BC307, U1 CR2013-MI2120, U2 RP2040-Zero, U3 L7805, U4 LDO-3.3, U5 Adafruit_MCP9600_Breakout, U6 Adafruit_MCP9600_Breakout, U7 MCP2515_CAN, U8 LDO-3.3, U9 GY_NEO6MV2

Commit message: feat(clocks): integrate oil pressure, ABS speed and EGT monitoring
-Split CAN and gauge control from display and sensor work across both cores
-Add charge lamp control and measurement validity handling in ECU and OBD
-Update HAL, hardware configuration, tests and docs
Parts:
- removed D3: 1N4007, Diode_THT:D_DO-41_SOD81_P10.16mm_Horizontal, symbol Diode:1N4007
Changed lines of the file:
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@@
 	)
 	(junction
-		(at 73.66 144.78)
-		(diameter 0)
-		(color 0 0 0 0)
-	)
-	(junction
 		(at 82.55 96.52)
 		(diameter 0)
@@
 	(wire
 		(pts
-			(xy 88.9 46.99) (xy 96.52 46.99)
-		)
-		(stroke
-			(width 0)
-			(type default)
-		)
-	)
-	(wire
-		(pts
 			(xy 130.81 130.81) (xy 133.35 130.81)
 		)
@@
 	(wire
 		(pts
-			(xy 48.26 46.99) (xy 81.28 46.99)
-		)
-		(stroke
-			(width 0)
-			(type default)
-		)
-	)
-	(wire
-		(pts
 			(xy 113.03 72.39) (xy 113.03 83.82)
 		)
@@
 	(wire
 		(pts
-			(xy 48.26 144.78) (xy 73.66 144.78)
-		)
-		(stroke
-			(width 0)
-			(type default)
-		)
-	)
-	(wire
-		(pts
 			(xy 179.07 71.12) (xy 200.66 71.12)
 		)
@@
 	(wire
 		(pts
-			(xy 48.26 46.99) (xy 48.26 144.78)
-		)
-		(stroke
-			(width 0)
-			(type default)
-		)
-	)
-	(wire
-		(pts
 			(xy 189.23 78.74) (xy 200.66 78.74)
 		)
@@
 					(unit 1)
 				)
-			)
-		)
-	)
-	(symbol
-		(lib_id "Diode:1N4007")
-		(at 85.09 46.99 0)
-		(unit 1)
-		(exclude_from_sim no)
-		(in_bom yes)
-		(on_board yes)
-		(dnp no)
-		(fields_autoplaced yes)
-		(property "Reference" "D3"
-			(at 85.09 40.64 0)
-			(effects
-				(font
-					(size 1.27 1.27)
-				)
-			)
-		)
-		(property "Value" "1N4007"
-			(at 85.09 43.18 0)
-			(effects
-				(font
-					(size 1.27 1.27)
-				)
-			)
-		)
-		(property "Footprint" "Diode_THT:D_DO-41_SOD81_P10.16mm_Horizontal"
-			(at 85.09 51.435 0)
-			(effects
-				(font
-					(size 1.27 1.27)
-				)
-				(hide yes)
-			)
-		)
-		(property "Datasheet" "http://www.vishay.com/docs/88503/1n4001.pdf"
-			(at 85.09 46.99 0)
-			(effects
-				(font
-					(size 1.27 1.27)
-				)
-				(hide yes)
-			)
-		)
-		(property "Description" "1000V 1A General Purpose Rectifier Diode, DO-41"
-			(at 85.09 46.99 0)
-			(effects
-				(font
-					(size 1.27 1.27)
-				)
-				(hide yes)
-			)
-		)
-		(property "Sim.Device" "D"
-			(at 85.09 46.99 0)
-			(effects
-				(font
-					(size 1.27 1.27)
-				)
-				(hide yes)
-			)
-		)
-		(property "Sim.Pins" "1=K 2=A"
-			(at 85.09 46.99 0)
-			(effects
-				(font
-					(size 1.27 1.27)
-				)
-				(hide yes)
-			)
-		)
-		(pin "2"
-		)
-		(pin "1"
-		)
-		(instances
-			(project "Clocks"
-				(path "/d7cff82a-6fa9-4f72-9c9c-4cac4f2ba6d5"
-					(reference "D3")
-					(unit 1)
-				)

Commit message: feat(fiesta_clock): synchronize RTC with GPS UTC
-Add verified RTC synchronization, persistent UTC tracking and CET/CEST editing
-Update HAL, share UTC CAN encoding and cover clock behavior with regression tests
-Update dashboard hardware files and remove unused fuel gauge code
Parts:
- added C10: 4,7uF, symbol Device:C_Polarized_Small
Connections:
- net GND: now also C10.2
- net at J3.6 (Pin_6), R14.2, U2.4 (GP29): now also C10.1
Changed lines of the file:
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@@
 	)
 	(junction
+		(at 113.03 83.82)
+		(diameter 0)
+		(color 0 0 0 0)
+	)
+	(junction
 		(at 187.96 107.95)
 		(diameter 0)
@@
 	(wire
 		(pts
+			(xy 107.95 83.82) (xy 107.95 85.09)
+		)
+		(stroke
+			(width 0)
+			(type default)
+		)
+	)
+	(wire
+		(pts
 			(xy 124.46 91.44) (xy 125.73 91.44)
 		)
@@
 	(wire
 		(pts
+			(xy 113.03 83.82) (xy 107.95 83.82)
+		)
+		(stroke
+			(width 0)
+			(type default)
+		)
+	)
+	(wire
+		(pts
 			(xy 127 142.24) (xy 146.05 142.24)
 		)
@@
 	(symbol
 		(lib_id "power:GND")
+		(at 107.95 90.17 0)
+		(unit 1)
+		(exclude_from_sim no)
+		(in_bom yes)
+		(on_board yes)
+		(dnp no)
+		(fields_autoplaced yes)
+		(property "Reference" "#PWR034"
+			(at 107.95 96.52 0)
+			(effects
+				(font
+					(size 1.27 1.27)
+				)
+				(hide yes)
+			)
+		)
+		(property "Value" "GND"
+			(at 107.9499 93.98 90)
+			(effects
+				(font
+					(size 1.27 1.27)
+				)
+				(justify right)
+				(hide yes)
+			)
+		)
+		(property "Footprint" ""
+			(at 107.95 90.17 0)
+			(effects
+				(font
+					(size 1.27 1.27)
+				)
+				(hide yes)
+			)
+		)
+		(property "Datasheet" ""
+			(at 107.95 90.17 0)
+			(effects
+				(font
+					(size 1.27 1.27)
+				)
+				(hide yes)
+			)
+		)
+		(property "Description" "Power symbol creates a global label with name \"GND\" , ground"
+			(at 107.95 90.17 0)
+			(effects
+				(font
+					(size 1.27 1.27)
+				)
+				(hide yes)
+			)
+		)
+		(pin "1"
+		)
+		(instances
+			(project "Clocks"
+				(path "/d7cff82a-6fa9-4f72-9c9c-4cac4f2ba6d5"
+					(reference "#PWR034")
+					(unit 1)
+				)
+			)
+		)
+	)
+	(symbol
+		(lib_id "power:GND")
 		(at 130.81 130.81 0)
 		(unit 1)
@@
 					(unit 1)
 				)
+			)
+		)
+	)
+	(symbol
+		(lib_id "Device:C_Polarized_Small")
+		(at 107.95 87.63 0)
+		(unit 1)
+		(exclude_from_sim no)
+		(in_bom yes)
+		(on_board yes)
+		(dnp no)
+		(property "Reference" "C10"
+			(at 110.49 85.8138 0)
+			(effects
+				(font
+					(size 1.27 1.27)
+				)
+				(justify left)
+				(hide yes)
+			)
+		)
+		(property "Value" "4,7uF"
+			(at 108.458 85.598 0)
+			(effects
+				(font
+					(size 1.27 1.27)
+				)
+				(justify left)
+			)
+		)
+		(property "Footprint" ""
+			(at 107.95 87.63 0)
+			(effects
+				(font
+					(size 1.27 1.27)
+				)
+				(hide yes)
+			)
+		)
+		(property "Datasheet" "~"
+			(at 107.95 87.63 0)
+			(effects
+				(font
+					(size 1.27 1.27)
+				)
+				(hide yes)
+			)
+		)
+		(property "Description" "Polarized capacitor, small symbol"
+			(at 107.95 87.63 0)
+			(effects
+				(font
+					(size 1.27 1.27)
+				)
+				(hide yes)
+			)
+		)
+		(pin "2"
+		)
+		(pin "1"
+		)
+		(instances
+			(project "Clocks"
+				(path "/d7cff82a-6fa9-4f72-9c9c-4cac4f2ba6d5"
+					(reference "C10")
+					(unit 1)
+				)
